File: rgb-tiles.kicad_pcb (KiCad board)
At the start: 2 copper layers, 99.5 x 99.5 mm, 247 parts, among them J1 SWD, J10 S POWER LINK, J11 W POWER LINK, J2 N / M20-8890645R, J3 E / M20-7910642R, J4 S / M20-7910642R, J5 W / M20-8890645R, J6 USB4110-GF-A, J7 12V INPUT, J8 N POWER LINK, J9 E POWER LINK, Q1 AO3400A, SW1 BOOT, SW2 RESET, U1 RP2040, U10 SN74AHCT1G125DBVR, U11 TPD2E2U06DCKR, U12 TPD2E2U06DCKR, U13 TPD2E2U06DCKR, U14 TPD2E2U06DCKR, U15 TPS26600PWPR, U2 W25Q16JVSSIQ, U3 AP63205WU-7, U4 AP2112K-3.3TRG1, U5 SN74LVC2G125DCUR, U6 SN74LVC2G125DCUR, U7 SN74LVC2G125DCUR, U8 SN74LVC2G125DCUR, U9 USBLC6-2SC6, Y1 ABM8-272-T3 12MHz

Commit message: finish tile routing and four-layer power layout
Parts:
- C103, C14: moved to F.Cu
- moved R25 20.7 mm to (82.3, 111.0)
- moved R26 20.6 mm to (80.4, 111.0)
- moved C13 11.8 mm to (78.0, 111.5), turned to 90 degrees
- moved U9 9.81 mm to (62.2, 137.9), turned to 90 degrees
- moved C103 6.36 mm to (80.8, 114.5), turned to 0 degrees
- moved F3 6.10 mm to (134.5, 106.0)
- moved R3 6.10 mm to (77.0, 130.6)
- moved C5 6.00 mm to (77.0, 123.3)
- moved C12 5.39 mm to (72.0, 111.0), turned to -90 degrees
- moved C16 4.74 mm to (128.5, 114.0)
- moved C10 3.51 mm to (87.5, 111.3)
- moved C11 3.36 mm to (90.1, 110.2)
- moved Y1 3.20 mm to (83.5, 124.8)
- moved R6 3.16 mm to (127.0, 108.0)
- moved C9 3.00 mm to (84.0, 111.5)
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Routing:
- net +3V3: track 0.00 -> 395.6 mm, vias 0 -> 15
- net +12V_BUS: track 0.00 -> 182.1 mm, vias 0 -> 10
- net LINK_DISABLE: track 0.00 -> 167.5 mm, vias 0 -> 13
- net GND: track 0.00 -> 113.8 mm, vias 0 -> 133
- net +5V: track 187.2 -> 276.5 mm, vias 0 -> 74
- net LED_DATA_3V3: track 0.00 -> 83.9 mm, vias 0 -> 3
- net N_TX: track 0.00 -> 66.5 mm, vias 0 -> 4
- net N_RX: track 0.00 -> 64.2 mm, vias 0 -> 3
- net W_RX: track 0.00 -> 59.4 mm, vias 0 -> 6
- net E_RX: track 0.00 -> 51.3 mm, vias 0 -> 2
- net W_TX: track 0.00 -> 48.8 mm, vias 0 -> 7
- net E_TX: track 0.00 -> 47.8 mm, vias 0 -> 2
- net USB_DM_ESD: track 0.00 -> 45.6 mm, vias 0 -> 2
- net USB_DP_ESD: track 0.00 -> 45.3 mm
- net USB_VBUS_N: track 0.00 -> 42.5 mm
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- added copper zone on In1.Cu, net +5V
- added copper zone on B.Cu, net EFUSE_RTN
- added copper zone on F.Cu, net EFUSE_RTN
- added copper zone on In1.Cu, net EFUSE_RTN
- added copper zone on In2.Cu, net EFUSE_RTN
- added copper zone on B.Cu, net GND
- added copper zone on F.Cu, net GND
- added copper zone on In1.Cu, net GND
- added copper zone on In2.Cu, net GND
Other:
- copper layers 2 -> 4

Commit message: add firmware, controller and manufacturing files
Parts:
- D70: value SS34 -> B340A
- U11, U12, U13, U14: value TPD2E2U06DCKR -> TPD2E2U06QDCKRQ1
