File: schematic/controller.kicad_sch (KiCad schematic)
At the start: 24 parts, among them J1 SWD, SW1 BOOT, SW2 RESET, U1 RP2040, U2 W25Q16JVSSIQ, Y1 ABM8-272-T3 12MHz

Commit message: finish tile schematics and connector footprints
Parts:
- added C103, C104: 100n 25V X7R, Capacitor_SMD:C_0603_1608Metric, symbol Device:C
- added TP6: +1V1, TestPoint:TestPoint_Pad_D1.5mm, symbol Connector:TestPoint
- C1, C2: value 15p -> 15p 50V C0G; MPN (none) -> C0603C150J5GACTU; Manufacturer (none) -> KEMET
- C10, C11, C14, C3, C4, C5, C6, C7, C8, C9: value 100n -> 100n 25V X7R; MPN (none) -> C0603C104K3RACTU; Manufacturer (none) -> KEMET
- C12, C13: value 1u -> 2.2u 16V X7R; footprint Capacitor_SMD:C_0603_1608Metric -> Capacitor_SMD:C_0805_2012Metric; MPN (none) -> C0805C225K4RACTU; Manufacturer (none) -> KEMET
- J1: MPN (none) -> A2541WV-4P; Manufacturer (none) -> CJT
- R1, R3: MPN (none) -> RC0603FR-0710KL; Manufacturer (none) -> Yageo; Power (none) -> 0.1W; Tolerance (none) -> 1%
- R2, R4: MPN (none) -> RC0603FR-071KL; Manufacturer (none) -> Yageo; Power (none) -> 0.1W; Tolerance (none) -> 1%
- SW1, SW2: MPN (none) -> TL3342F160QG/TR; Manufacturer (none) -> E-Switch
- U1: MPN (none) -> RP2040; Manufacturer (none) -> Raspberry Pi
- U2: MPN (none) -> W25Q16JVSSIQ; Manufacturer (none) -> Winbond
- Y1: MPN (none) -> ABM8-272-T3; Manufacturer (none) -> Abracon
Connections:
- net +1V1: now also C103.1, TP6.1
- net +3V3: now also C104.1
- net GND: now also C103.2, C104.2
- net USB_VBUS_DETECT renamed USB_VBUS_N

Commit message: add firmware, controller and manufacturing files
Parts:
- C10, C103, C104, C11, C14, C3, C4, C5, C6, C7, C8, C9: MPN C0603C104K3RACTU -> CL10B104KA8NNNC; Manufacturer KEMET -> Samsung Electro-Mechanics
- J1: MPN A2541WV-4P -> TSW-104-07-T-S; Manufacturer CJT -> Samtec
- SW1, SW2: MPN TL3342F160QG/TR -> TL3342F160QG
- U2: MPN W25Q16JVSSIQ -> W25Q16JVSSIM
Changed lines of the file:
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@@
 			)
 		)
-		(property "MPN" "W25Q16JVSSIQ"
+		(property "MPN" "W25Q16JVSSIM"
 			(at 199.39 69.85 0)
 			(effects
@@
 			)
 		)
-		(property "MPN" "TL3342F160QG/TR"
+		(property "MPN" "TL3342F160QG"
 			(at 260.35 69.85 0)
 			(effects
@@
 			)
 		)
-		(property "MPN" "TL3342F160QG/TR"
+		(property "MPN" "TL3342F160QG"
 			(at 199.39 110.49 0)
 			(effects
@@
 			)
 		)
-		(property "Datasheet" "https://www.cjt.com/upload/A2541.pdf"
+		(property "Datasheet" "https://suddendocs.samtec.com/prints/tsw-xxx-xx-xxx-x-xx-xxx-mkt.pdf"
 			(at 345.44 64.77 0)
 			(effects
@@
 			)
 		)
-		(property "Manufacturer" "CJT"
+		(property "Manufacturer" "Samtec"
 			(at 345.44 64.77 0)
 			(effects
@@
 			)
 		)
-		(property "MPN" "A2541WV-4P"
+		(property "MPN" "TSW-104-07-T-S"
 			(at 345.44 64.77 0)
 			(effects
@@
 			)
 		)
-		(property "Datasheet" "https://search.kemet.com/component-documentation/download/specsheet/C0603C104K3RACTU"
+		(property "Datasheet" "https://product.samsungsem.com/mlcc/CL10B104KA8NNN.do"
 			(at 30.48 209.55 0)
 			(effects
@@
 			)
 		)
-		(property "Manufacturer" "KEMET"
+		(property "Manufacturer" "Samsung Electro-Mechanics"
 			(at 30.48 209.55 0)
 			(effects
@@
 			)
 		)
-		(property "MPN" "C0603C104K3RACTU"
+		(property "MPN" "CL10B104KA8NNNC"
 			(at 30.48 209.55 0)
 			(effects
@@
 			)
 		)
-		(property "Datasheet" "https://search.kemet.com/component-documentation/download/specsheet/C0603C104K3RACTU"
+		(property "Datasheet" "https://product.samsungsem.com/mlcc/CL10B104KA8NNN.do"
 			(at 67.31 209.55 0)
 			(effects
@@
 			)
 		)
-		(property "Manufacturer" "KEMET"
+		(property "Manufacturer" "Samsung Electro-Mechanics"
 			(at 67.31 209.55 0)
 			(effects
@@
 			)
 		)
-		(property "MPN" "C0603C104K3RACTU"
+		(property "MPN" "CL10B104KA8NNNC"
 			(at 67.31 209.55 0)
 			(effects
@@
 			)
 		)
-		(property "Datasheet" "https://search.kemet.com/component-documentation/download/specsheet/C0603C104K3RACTU"
+		(property "Datasheet" "https://product.samsungsem.com/mlcc/CL10B104KA8NNN.do"
 			(at 104.14 209.55 0)
 			(effects
@@
 			)
 		)
-		(property "Manufacturer" "KEMET"
+		(property "Manufacturer" "Samsung Electro-Mechanics"
 			(at 104.14 209.55 0)
 			(effects
@@
 			)
 		)
-		(property "MPN" "C0603C104K3RACTU"
+		(property "MPN" "CL10B104KA8NNNC"
 			(at 104.14 209.55 0)
 			(effects
@@
 			)
 		)
-		(property "Datasheet" "https://search.kemet.com/component-documentation/download/specsheet/C0603C104K3RACTU"
+		(property "Datasheet" "https://product.samsungsem.com/mlcc/CL10B104KA8NNN.do"
 			(at 140.97 209.55 0)
 			(effects
@@
 			)
 		)
-		(property "Manufacturer" "KEMET"
+		(property "Manufacturer" "Samsung Electro-Mechanics"
 			(at 140.97 209.55 0)
 			(effects
@@
 			)
 		)
-		(property "MPN" "C0603C104K3RACTU"
+		(property "MPN" "CL10B104KA8NNNC"
 			(at 140.97 209.55 0)
 			(effects
@@
 			)
 		)
-		(property "Datasheet" "https://search.kemet.com/component-documentation/download/specsheet/C0603C104K3RACTU"
+		(property "Datasheet" "https://product.samsungsem.com/mlcc/CL10B104KA8NNN.do"
 			(at 177.8 209.55 0)
 			(effects
@@
 			)
 		)
-		(property "Manufacturer" "KEMET"
+		(property "Manufacturer" "Samsung Electro-Mechanics"
 			(at 177.8 209.55 0)
 			(effects
@@
 			)
 		)
-		(property "MPN" "C0603C104K3RACTU"
+		(property "MPN" "CL10B104KA8NNNC"
 			(at 177.8 209.55 0)
 			(effects
@@
 			)
 		)
-		(property "Datasheet" "https://search.kemet.com/component-documentation/download/specsheet/C0603C104K3RACTU"
+		(property "Datasheet" "https://product.samsungsem.com/mlcc/CL10B104KA8NNN.do"
 			(at 214.63 209.55 0)
 			(effects
@@
 			)
 		)
-		(property "Manufacturer" "KEMET"
+		(property "Manufacturer" "Samsung Electro-Mechanics"
 			(at 214.63 209.55 0)
 			(effects
@@
 			)
 		)
-		(property "MPN" "C0603C104K3RACTU"
+		(property "MPN" "CL10B104KA8NNNC"
 			(at 214.63 209.55 0)
 			(effects
@@
 			)
 		)
-		(property "Datasheet" "https://search.kemet.com/component-documentation/download/specsheet/C0603C104K3RACTU"
+		(property "Datasheet" "https://product.samsungsem.com/mlcc/CL10B104KA8NNN.do"
 			(at 251.46 209.55 0)
 			(effects
@@
 			)
 		)
-		(property "Manufacturer" "KEMET"
+		(property "Manufacturer" "Samsung Electro-Mechanics"
 			(at 251.46 209.55 0)
 			(effects
@@
 			)
 		)
-		(property "MPN" "C0603C104K3RACTU"
+		(property "MPN" "CL10B104KA8NNNC"
 			(at 251.46 209.55 0)
 			(effects
@@
 			)
 		)
-		(property "Datasheet" "https://search.kemet.com/component-documentation/download/specsheet/C0603C104K3RACTU"
+		(property "Datasheet" "https://product.samsungsem.com/mlcc/CL10B104KA8NNN.do"
 			(at 289.56 209.55 0)
 			(effects
@@
 			)
 		)
-		(property "Manufacturer" "KEMET"
+		(property "Manufacturer" "Samsung Electro-Mechanics"
 			(at 289.56 209.55 0)
 			(effects
@@
 			)
 		)
-		(property "MPN" "C0603C104K3RACTU"
+		(property "MPN" "CL10B104KA8NNNC"
 			(at 289.56 209.55 0)
 			(effects
@@
 			)
 		)
-		(property "Datasheet" "https://search.kemet.com/component-documentation/download/specsheet/C0603C104K3RACTU"
+		(property "Datasheet" "https://product.samsungsem.com/mlcc/CL10B104KA8NNN.do"
 			(at 326.39 209.55 0)
 			(effects
@@
 			)
 		)
-		(property "Manufacturer" "KEMET"
+		(property "Manufacturer" "Samsung Electro-Mechanics"
 			(at 326.39 209.55 0)
 			(effects
@@
 			)
 		)
-		(property "MPN" "C0603C104K3RACTU"
+		(property "MPN" "CL10B104KA8NNNC"
 			(at 326.39 209.55 0)
 			(effects
@@
 			)
 		)
-		(property "Datasheet" "https://search.kemet.com/component-documentation/download/specsheet/C0603C104K3RACTU"
+		(property "Datasheet" "https://product.samsungsem.com/mlcc/CL10B104KA8NNN.do"
 			(at 180.34 250.19 0)
 			(effects
@@
 			)
 		)
-		(property "Manufacturer" "KEMET"
+		(property "Manufacturer" "Samsung Electro-Mechanics"
 			(at 180.34 250.19 0)
 			(effects
@@
 			)
 		)
-		(property "MPN" "C0603C104K3RACTU"
+		(property "MPN" "CL10B104KA8NNNC"
 			(at 180.34 250.19 0)
 			(effects
@@
 			)
 		)
-		(property "Datasheet" "https://search.kemet.com/component-documentation/download/specsheet/C0603C104K3RACTU"
+		(property "Datasheet" "https://product.samsungsem.com/mlcc/CL10B104KA8NNN.do"
 			(at 240.03 250.19 0)
 			(effects
@@
 			)
 		)
-		(property "Manufacturer" "KEMET"
+		(property "Manufacturer" "Samsung Electro-Mechanics"
 			(at 240.03 250.19 0)
 			(effects
@@
 			)
 		)
-		(property "MPN" "C0603C104K3RACTU"
+		(property "MPN" "CL10B104KA8NNNC"
 			(at 240.03 250.19 0)
 			(effects
@@
 			)
 		)
-		(property "Datasheet" "https://search.kemet.com/component-documentation/download/specsheet/C0603C104K3RACTU"
+		(property "Datasheet" "https://product.samsungsem.com/mlcc/CL10B104KA8NNN.do"
 			(at 363.22 209.55 0)
 			(effects
@@
 			)
 		)
-		(property "Manufacturer" "KEMET"
+		(property "Manufacturer" "Samsung Electro-Mechanics"
 			(at 363.22 209.55 0)
 			(effects
@@
 			)
 		)
-		(property "MPN" "C0603C104K3RACTU"
+		(property "MPN" "CL10B104KA8NNNC"
 			(at 363.22 209.55 0)
 			(effects
