File: schematic/power-inlet.kicad_sch (KiCad schematic)
At the start: 9 parts, among them J7 12V INPUT, U15 TPS26600PWPR

Commit message: place tile components and route led data chain
Parts:
- U15: footprint Package_SO:HTSSOP-16-1EP_4.4x5mm_P0.65mm_EP3.4x5mm_Mask2.66x2.46mm_ThermalVias -> RGB_Tiles:HTSSOP16_EP_4.4x5_P0.65_Vias0.3
Changed lines of the file:
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@@
 			)
 		)
-		(property "Footprint" "Package_SO:HTSSOP-16-1EP_4.4x5mm_P0.65mm_EP3.4x5mm_Mask2.66x2.46mm_ThermalVias"
+		(property "Footprint" "RGB_Tiles:HTSSOP16_EP_4.4x5_P0.65_Vias0.3"
 			(at 110.49 105.41 0)
 			(effects

Commit message: add firmware, controller and manufacturing files
Parts:
- D70: value SS34 -> B340A; MPN SS34-13-F -> B340A-13-F
Changed lines of the file:
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@@
 			)
 		)
-		(property "Value" "SS34"
+		(property "Value" "B340A"
 			(at 335.28 97.79 0)
 			(effects
@@
 			)
 		)
-		(property "Datasheet" "https://www.diodes.com/part/view/SS34"
+		(property "Datasheet" "https://www.diodes.com/datasheet/download/B340A.pdf"
 			(at 335.28 95.25 0)
 			(effects
@@
 			)
 		)
-		(property "MPN" "SS34-13-F"
+		(property "MPN" "B340A-13-F"
 			(at 335.28 95.25 0)
 			(effects
