File: schematic/usb-led-data.kicad_sch (KiCad schematic)
At the start: 13 parts, among them J6 USB-C, U10 SN74AHCT1G125DBVR, U9 USBLC6-2SC6

Commit message: finish tile schematics and connector footprints
Parts:
- added Q1: AO3400A, Package_TO_SOT_SMD:SOT-23, symbol Transistor_FET:AO3400A
- added R35: 10k, Resistor_SMD:R_0603_1608Metric, symbol Device:R
- added TP7: LED DATA, TestPoint:TestPoint_Pad_D1.5mm, symbol Connector:TestPoint
- added TP8: VBUS, TestPoint:TestPoint_Pad_D1.5mm, symbol Connector:TestPoint
- C94, C95: value 100n -> 100n 25V X7R; MPN (none) -> C0603C104K3RACTU; Manufacturer (none) -> KEMET
- J6: value USB-C -> USB4105-GF-A; MPN (none) -> USB4105-GF-A; Manufacturer (none) -> GCT
- R23, R24: MPN (none) -> RC0603FR-075K1L; Manufacturer (none) -> Yageo; Power (none) -> 0.1W; Tolerance (none) -> 1%
- R25, R26: MPN (none) -> RC0603FR-0727RL; Manufacturer (none) -> Yageo; Power (none) -> 0.1W; Tolerance (none) -> 1%
- R27, R29: MPN (none) -> RC0603FR-07100KL; Manufacturer (none) -> Yageo; Power (none) -> 0.1W; Tolerance (none) -> 1%
- R28: value 100k -> 1M; MPN (none) -> RC0603FR-071ML; Manufacturer (none) -> Yageo; Power (none) -> 0.1W; Tolerance (none) -> 1%
- R30: MPN (none) -> RC0603FR-07100RL; Manufacturer (none) -> Yageo; Power (none) -> 0.1W; Tolerance (none) -> 1%
- U10: footprint (none) -> Package_TO_SOT_SMD:SOT-23-5; MPN (none) -> SN74AHCT1G125DBVR; Manufacturer (none) -> Texas Instruments
- U9: MPN (none) -> USBLC6-2SC6; Manufacturer (none) -> STMicroelectronics
Connections:
- net GND: now also Q1.2 (S)
- net LED_DATA_5V: now also TP7.1
- net USB_VBUS: now also TP8.1
- net USB_VBUS_DETECT renamed USB_DETECT_GATE
- net USB_DETECT_GATE: now also Q1.1 (G)
- new net +3V3: R35.1
- new net USB_VBUS_N: Q1.3 (D), R35.2
Other:
- moved on the sheet: C94, R27

Commit message: place tile components and route led data chain
Parts:
- J6: value USB4105-GF-A -> USB4110-GF-A; footprint Connector_USB:USB_C_Receptacle_GCT_USB4105-xx-A_16P_TopMnt_Horizontal -> Connector_USB:USB_C_Receptacle_GCT_USB4110; MPN USB4105-GF-A -> USB4110-GF-A
Changed lines of the file:
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@@
 			)
 		)
-		(property "Value" "USB4105-GF-A"
+		(property "Value" "USB4110-GF-A"
 			(at 44.45 45.085 0)
 			(effects
@@
 			)
 		)
-		(property "Footprint" "Connector_USB:USB_C_Receptacle_GCT_USB4105-xx-A_16P_TopMnt_Horizontal"
+		(property "Footprint" "Connector_USB:USB_C_Receptacle_GCT_USB4110"
 			(at 44.45 64.77 0)
 			(effects
@@
 			)
 		)
-		(property "Datasheet" "https://gct.co/download?name=USB4105.pdf&type=PDFDrawing"
+		(property "Datasheet" "https://gct.co/download?name=USB4110.pdf&type=PDFDrawing"
 			(at 44.45 64.77 0)
 			(effects
@@
 			)
 		)
-		(property "MPN" "USB4105-GF-A"
+		(property "MPN" "USB4110-GF-A"
 			(at 44.45 64.77 0)
 			(effects

Commit message: add firmware, controller and manufacturing files
Parts:
- C94, C95: MPN C0603C104K3RACTU -> CL10B104KA8NNNC; Manufacturer KEMET -> Samsung Electro-Mechanics
Changed lines of the file:
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@@
 			)
 		)
-		(property "Datasheet" "https://search.kemet.com/component-documentation/download/specsheet/C0603C104K3RACTU"
+		(property "Datasheet" "https://product.samsungsem.com/mlcc/CL10B104KA8NNN.do"
 			(at 299.72 124.46 0)
 			(effects
@@
 			)
 		)
-		(property "Manufacturer" "KEMET"
+		(property "Manufacturer" "Samsung Electro-Mechanics"
 			(at 299.72 124.46 0)
 			(effects
@@
 			)
 		)
-		(property "MPN" "C0603C104K3RACTU"
+		(property "MPN" "CL10B104KA8NNNC"
 			(at 299.72 124.46 0)
 			(effects
@@
 			)
 		)
-		(property "Datasheet" "https://search.kemet.com/component-documentation/download/specsheet/C0603C104K3RACTU"
+		(property "Datasheet" "https://product.samsungsem.com/mlcc/CL10B104KA8NNN.do"
 			(at 110.49 250.19 0)
 			(effects
@@
 			)
 		)
-		(property "Manufacturer" "KEMET"
+		(property "Manufacturer" "Samsung Electro-Mechanics"
 			(at 110.49 250.19 0)
 			(effects
@@
 			)
 		)
-		(property "MPN" "C0603C104K3RACTU"
+		(property "MPN" "CL10B104KA8NNNC"
 			(at 110.49 250.19 0)
 			(effects
